File: Dragon32_MKII.kicad_pcb (KiCad board)
At the start: 2 copper layers, 253 x 169.1 mm, 215 parts, among them IC1 4116, IC10 SFC2318, IC11 4053, IC12 6847, IC13 74LS273, IC14 74LS86, IC15 74LS783, IC16 74LS244, IC17 ROM8K, IC18 ROM8K, IC19 6809E, IC2 4116, IC20 4529, IC21 74LS123, IC22 74LS00, IC23 74LS74, IC24 74LS244, IC25 LM393, IC26 6821, IC27 74LS20, IC28 74LS393, IC29 74LS393, IC3 4116, IC30 74LS32, IC31 74LS02, IC32 74LS390, IC33 74LS138, IC34 4050, IC35 6821, IC36 4116, IC37 4116, IC38 4116, IC39 4116, IC4 4116, IC40 4116, IC41 4116, IC42 4116, IC43 4116, IC5 4116, IC6 4116, IC7 4116, IC8 4116, IC9 LM1889, SW1 RESET

Commit message: align component positions to board
Parts:
- C71: footprint Capacitor_THT:C_Disc_D4.3mm_W1.9mm_P5.00mm -> Capacitor_THT:C_Disc_D3.8mm_W2.6mm_P2.50mm
- D11: footprint Diode_THT:D_DO-35_SOD27_P7.62mm_Horizontal -> Diode_THT:D_DO-35_SOD27_P10.16mm_Horizontal
- moved C50 421.6 mm to (321.8, 69.0), turned to 90 degrees
- moved C49 413.3 mm to (312.0, 62.0)
- moved R14 403.1 mm to (309.9, 92.7)
- moved R13 402.0 mm to (309.9, 95.8)
- moved C60 398.2 mm to (313.2, 88.1)
- moved D11 397.3 mm to (320.0, 98.6), turned to 180 degrees
- moved C21 394.0 mm to (299.3, 62.0)
- moved C19 387.8 mm to (274.1, 62.0)
- moved R40 386.9 mm to (324.9, 169.2), turned to -90 degrees
- moved C58 384.9 mm to (300.5, 88.6)
- moved C20 380.9 mm to (286.6, 62.0)
- moved C18 374.4 mm to (261.2, 62.0)
- moved C70 372.4 mm to (297.4, 91.5), turned to -90 degrees
- moved C73 371.5 mm to (297.4, 105.6), turned to 90 degrees
- moved C57 370.6 mm to (286.6, 88.4)
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Connections:
- D11 pad 1: ~{HALT} -> ~{RES}
- D11 pad 2: ~{RES} -> ~{HALT}

Commit message: more layout
Parts:
- D11: footprint Diode_THT:D_DO-35_SOD27_P10.16mm_Horizontal -> Diode_THT:D_DO-35_SOD27_P12.70mm_Horizontal
- R1, R10, R11, R12, R13, R14, R15, R16, R17, R18, R19, R2, R20, R21, R22, R23, R24, R25, R26, R27, R28, R29, R3, R30, R31, R32, R33, R34, R35, R36, R37, R38, R39, R4, R40, R41, R42, R43, R44, R45, R46, R47, R48, R49, R5, R50, R51, R52, R53, R54, R55, R56, R57, R58, R59, R6, R60, R61, R62, R63, R64, R65, R66, R67, R68, R69, R7, R70, R71, R72, R73, R8, R9: footprint Resistor_THT:R_Axial_DIN0207_L6.3mm_D2.5mm_P10.16mm_Horizontal -> Dragon:R_Axial_DIN0207_L6.3mm_D2.5mm_P12.7mm_Horizontal
- moved R72 365.0 mm to (321.8, 71.9), turned to -90 degrees
- moved R66 363.5 mm to (324.8, 71.9), turned to -90 degrees
- moved C68 356.1 mm to (287.8, 117.8)
- moved C67 343.1 mm to (275.2, 118.0)
- moved C66 329.8 mm to (262.3, 118.0)
- moved R25 322.1 mm to (247.6, 150.8), turned to 90 degrees
- moved C64 319.4 mm to (236.9, 118.1)
- moved R24 319.3 mm to (244.7, 150.7), turned to 90 degrees
- moved C65 316.9 mm to (249.9, 118.1)
- moved R23 316.5 mm to (241.7, 150.7), turned to 90 degrees
- moved R22 313.8 mm to (238.7, 150.7), turned to 90 degrees
- moved R21 311.1 mm to (235.8, 150.7), turned to 90 degrees
- moved R20 308.5 mm to (232.8, 150.7), turned to 90 degrees
- moved C63 306.4 mm to (224.4, 118.0)
- moved R19 306.0 mm to (229.9, 150.7), turned to 90 degrees
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
Commit message: position components
Parts:
- R10, R67, R68, R69, R70, R8, R9: footprint Dragon:R_Axial_DIN0207_L6.3mm_D2.5mm_P12.7mm_Horizontal -> Resistor_THT:R_Axial_DIN0207_L6.3mm_D2.5mm_P10.16mm_Horizontal
- moved C74 240.1 mm to (279.6, 159.4)
- moved R39 236.4 mm to (274.9, 164.5)
- moved R12 208.6 mm to (223.2, 155.4)
- moved D10 202.7 mm to (246.2, 163.0), turned to 90 degrees
- moved R38 186.7 mm to (223.4, 162.8)
- moved C72 177.2 mm to (216.6, 154.8), turned to -90 degrees
- moved R8 166.6 mm to (178.3, 79.9), turned to 90 degrees
- moved R9 164.6 mm to (175.3, 79.9), turned to 90 degrees
- moved R10 163.0 mm to (169.2, 69.7), turned to -90 degrees
- moved C45 160.9 mm to (177.6, 221.2)
- moved R11 151.0 mm to (159.6, 82.6)
- moved C4 149.0 mm to (132.2, 62.8), turned to -90 degrees
- moved R53 145.7 mm to (168.3, 209.3), turned to 90 degrees
- moved R55 145.5 mm to (174.4, 209.3), turned to 90 degrees
- moved R54 145.5 mm to (171.4, 209.3), turned to 90 degrees
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