File: Dragon32_MKII.kicad_sch (KiCad schematic)
At the start: 223 parts, among them IC1 4116, IC10 SFC2318, IC11 4053, IC12 6847, IC13 74LS273, IC14 74LS86, IC15 74LS783, IC16 74LS244, IC17 ROM8K, IC18 ROM8K, IC19 6809E, IC2 4116, IC20 4529, IC21 74LS123, IC22 74LS00, IC23 74LS74, IC24 74LS244, IC25 LM393, IC26 6821, IC27 74LS20, IC28 74LS393, IC29 74LS393, IC3 4116, IC30 74LS32, IC31 74LS02, IC32 74LS390, IC33 74LS138, IC34 4050, IC35 6821, IC36 4116, IC37 4116, IC38 4116, IC39 4116, IC4 4116, IC40 4116, IC41 4116, IC42 4116, IC43 4116, IC5 4116, IC6 4116, IC7 4116, IC8 4116, IC9 LM1889, SW1 RESET, U1 LINE_PULSE_DIAGRAM

Commit message: complete tracing
Parts:
- C13, C29: footprint Capacitor_THT:CP_Radial_D5.0mm_P2.50mm -> Capacitor_THT:CP_Radial_Tantal_D6.0mm_P5.00mm
Connections:
- net CASOUT: now also C26.2, R16.2; no longer C26.1, R16.1
- net GND: now also C26.1, R16.1; no longer C26.2, R16.2
- net MD1: no longer IC13.4 (D1)
- net MD2: now also IC13.4 (D1)
- net ~{RAS0}: now also R26.1; no longer R26.2
- net at IC15.12 (~{RAS0}): now also R26.2; no longer R26.1
- net at IC11.14 (Z): now also R6.1; no longer R6.2
- net at R10.2, R11.1, R65.1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: now also R6.2; no longer R6.1
Other:
- moved on the sheet: R26, R6
Changed lines of the file:
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@@
     (effects (font (size 1.27 1.27)) (justify left bottom))
   )
-  (label "MD1" (at 49.53 210.82 0) (fields_autoplaced)
+  (label "MD2" (at 49.53 210.82 0) (fields_autoplaced)
     (effects (font (size 1.27 1.27)) (justify left bottom))
   )
@@
     )
   )
-  (symbol (lib_id "Dragon32_MKII:R") (at 219.71 62.23 90) (unit 1)
+  (symbol (lib_id "Dragon32_MKII:R") (at 219.71 62.23 270) (mirror x) (unit 1)
     (in_bom yes) (on_board yes) (dnp no)
     (property "Reference" "R26" (at 219.71 62.23 90)
       (effects (font (size 1.27 1.27)))
     )
-    (property "Value" "22R" (at 228.6 60.96 90)
+    (property "Value" "22R" (at 210.82 60.96 90)
       (effects (font (size 1.27 1.27)) (justify left) hide)
     )
@@
     )
   )
-  (symbol (lib_id "Dragon32_MKII:R") (at 553.72 213.36 0) (unit 1)
+  (symbol (lib_id "Dragon32_MKII:R") (at 553.72 213.36 0) (mirror x) (unit 1)
     (in_bom yes) (on_board yes) (dnp no)
-    (property "Reference" "R16" (at 557.53 212.09 0)
+    (property "Reference" "R16" (at 557.53 214.63 0)
       (effects (font (size 1.27 1.27)))
     )
-    (property "Value" "33K" (at 557.53 214.63 0)
+    (property "Value" "33K" (at 557.53 212.09 0)
       (effects (font (size 1.27 1.27)))
     )
@@
     )
   )
-  (symbol (lib_id "Dragon32_MKII:C") (at 563.88 213.36 0) (unit 1)
+  (symbol (lib_id "Dragon32_MKII:C") (at 563.88 213.36 0) (mirror x) (unit 1)
     (in_bom yes) (on_board yes) (dnp no)
-    (property "Reference" "C26" (at 567.69 212.09 0)
+    (property "Reference" "C26" (at 567.69 214.63 0)
       (effects (font (size 1.27 1.27)) (justify left))
     )
-    (property "Value" "2nF" (at 567.69 214.63 0)
+    (property "Value" "2nF" (at 567.69 212.09 0)
       (effects (font (size 1.27 1.27)) (justify left))
     )
-    (property "Footprint" "Capacitor_THT:C_Disc_D4.3mm_W1.9mm_P5.00mm" (at 564.8452 217.17 0)
+    (property "Footprint" "Capacitor_THT:C_Disc_D4.3mm_W1.9mm_P5.00mm" (at 564.8452 209.55 0)
       (effects (font (size 0.762 0.762)) hide)
     )
@@
       (effects (font (size 1.27 1.27)) (justify left))
     )
-    (property "Footprint" "Capacitor_THT:CP_Radial_D5.0mm_P2.50mm" (at 468.63 347.98 0)
+    (property "Footprint" "Capacitor_THT:CP_Radial_Tantal_D6.0mm_P5.00mm" (at 468.63 347.98 0)
       (effects (font (size 1.524 1.524)) hide)
     )
@@
     )
   )
-  (symbol (lib_id "Dragon32_MKII:R") (at 449.58 361.95 270) (unit 1)
+  (symbol (lib_id "Dragon32_MKII:R") (at 449.58 361.95 90) (mirror x) (unit 1)
     (in_bom yes) (on_board yes) (dnp no)
     (property "Reference" "R6" (at 449.58 356.87 90)
@@
       (effects (font (size 1.27 1.27)) (justify left))
     )
-    (property "Footprint" "Capacitor_THT:CP_Radial_D5.0mm_P2.50mm" (at 575.31 360.68 0)
+    (property "Footprint" "Capacitor_THT:CP_Radial_Tantal_D6.0mm_P5.00mm" (at 575.31 360.68 0)
       (effects (font (size 1.524 1.524)) hide)
     )

Commit message: finish tracing with relay
Parts:
- removed RLA1: RELAY, Dragon:OJS HM 10A Relay, symbol Dragon32_MKII:RELAY
- added RLA1: SPDT, Relay_THT:Relay_SPDT_HJR-4102, symbol Relay:TIANBO-HJR-4102-L
- C10: footprint Capacitor_THT:CP_Radial_D5.0mm_P2.50mm -> Capacitor_THT:CP_Radial_Tantal_D5.5mm_P5.00mm
- C11: footprint Capacitor_THT:CP_Radial_D5.0mm_P2.50mm -> Capacitor_THT:CP_Radial_Tantal_D6.0mm_P5.00mm
- renumbered R21 to R20, R20 to R21, R24 to R23, R23 to R24
Connections:
- net +12V: now also RLA1.5
- net at C27.1, D3.2 (K), PL4.1: now also RLA1.1, RLA1.12
- net at C27.2, D2.2 (K), PL4.3: now also RLA1.6
- net at D1.1 (A), TR1.2 (C): now also RLA1.8
- no-connect marks 54 -> 55
Other:
- moved on the sheet: D1
Changed lines of the file:
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@@
   (junction (at 474.98 356.87) (diameter 0) (color 0 0 0 0)
   )
+  (junction (at 643.89 160.02) (diameter 0) (color 0 0 0 0)
+  )
   (junction (at 119.38 562.61) (diameter 0) (color 0 0 0 0)
   )
@@
   (junction (at 438.15 142.24) (diameter 0) (color 0 0 0 0)
   )
+  (junction (at 656.59 144.78) (diameter 0) (color 0 0 0 0)
+  )
   (junction (at 218.44 331.47) (diameter 0) (color 0 0 0 0)
   )
@@
   (junction (at 44.45 102.87) (diameter 0) (color 0 0 0 0)
   )
-  (junction (at 638.81 144.78) (diameter 0) (color 0 0 0 0)
+  (junction (at 629.92 144.78) (diameter 0) (color 0 0 0 0)
   )
   (junction (at 779.78 67.31) (diameter 0) (color 0 0 0 0)
@@
   (junction (at 553.72 167.64) (diameter 0) (color 0 0 0 0)
   )
-  (junction (at 648.97 144.78) (diameter 0) (color 0 0 0 0)
-  )
   (junction (at 450.85 149.86) (diameter 0) (color 0 0 0 0)
   )
@@
   (junction (at 277.622 554.99) (diameter 0) (color 0 0 0 0)
   )
-  (junction (at 648.97 160.02) (diameter 0) (color 0 0 0 0)
-  )
   (junction (at 492.76 349.25) (diameter 0) (color 0 0 0 0)
   )
@@
   (no_connect (at 518.16 288.29))
   (no_connect (at 518.16 285.75))
+  (no_connect (at 651.51 160.02))
   (no_connect (at 210.82 370.84))
   (no_connect (at 241.3 368.3))
@@
     (stroke (width 0) (type default))
   )
-  (wire (pts (xy 638.81 144.78) (xy 648.97 144.78))
-    (stroke (width 0) (type default))
-  )
   (wire (pts (xy 505.46 355.6) (xy 505.46 370.84))
     (stroke (width 0) (type default))
@@
     (stroke (width 0) (type default))
   )
-  (wire (pts (xy 638.81 157.48) (xy 638.81 160.02))
+  (wire (pts (xy 629.92 157.48) (xy 629.92 160.02))
     (stroke (width 0) (type default))
   )
@@
     (stroke (width 0) (type default))
   )
-  (wire (pts (xy 453.39 374.65) (xy 455.93 374.65))
+  (wire (pts (xy 643.89 160.02) (xy 648.97 160.02))
     (stroke (width 0) (type default))
   )
-  (wire (pts (xy 144.78 181.61) (xy 140.97 181.61))
+  (wire (pts (xy 453.39 374.65) (xy 455.93 374.65))
     (stroke (width 0) (type default))
   )
-  (wire (pts (xy 648.97 160.02) (xy 648.97 162.56))
+  (wire (pts (xy 144.78 181.61) (xy 140.97 181.61))
     (stroke (width 0) (type default))
   )
@@
     (stroke (width 0) (type default))
   )
+  (wire (pts (xy 648.97 160.02) (xy 648.97 162.56))
+    (stroke (width 0) (type default))
+  )
   (wire (pts (xy 219.71 440.69) (xy 224.79 440.69))
     (stroke (width 0) (type default))
@@
     (stroke (width 0) (type default))
   )
+  (wire (pts (xy 629.92 144.78) (xy 643.89 144.78))
+    (stroke (width 0) (type default))
+  )
   (bus (pts (xy 278.13 431.8) (xy 275.59 431.8))
     (stroke (width 0) (type default))
@@
     (stroke (width 0) (type default))
   )
-  (wire (pts (xy 648.97 144.78) (xy 650.24 144.78))
-    (stroke (width 0) (type default))
-  )
   (bus (pts (xy 449.58 78.74) (xy 449.58 81.28))
     (stroke (width 0) (type default))
@@
     (stroke (width 0) (type default))
   )
-  (wire (pts (xy 638.81 147.32) (xy 638.81 144.78))
+  (wire (pts (xy 629.92 147.32) (xy 629.92 144.78))
     (stroke (width 0) (type default))
   )
@@
     (stroke (width 0) (type default))
   )
-  (wire (pts (xy 637.54 144.78) (xy 638.81 144.78))
+  (wire (pts (xy 628.65 144.78) (xy 629.92 144.78))
     (stroke (width 0) (type default))
   )
@@
     (stroke (width 0) (type default))
   )
+  (wire (pts (xy 654.05 144.78) (xy 656.59 144.78))
+    (stroke (width 0) (type default))
+  )
   (wire (pts (xy 228.6 64.77) (xy 223.52 64.77))
     (stroke (width 0) (type default))
@@
     (stroke (width 0) (type default))
   )
-  (wire (pts (xy 648.97 160.02) (xy 638.81 160.02))
+  (wire (pts (xy 629.92 160.02) (xy 643.89 160.02))
     (stroke (width 0) (type default))
   )
@@
     (effects (font (size 1.27 1.27)) (justify left bottom))
   )
-  (label "+12V" (at 641.35 144.78 0) (fields_autoplaced)
+  (label "+12V" (at 632.46 144.78 0) (fields_autoplaced)
     (effects (font (size 1.27 1.27)) (justify left bottom))
   )
@@
   (symbol (lib_id "Dragon32_MKII:R") (at 219.71 39.37 90) (unit 1)
     (in_bom yes) (on_board yes) (dnp no)
-    (property "Reference" "R24" (at 219.71 39.37 90)
+    (property "Reference" "R23" (at 219.71 39.37 90)
       (effects (font (size 1.27 1.27)))
     )
@@
       (project "Dragon32_MKII"
         (path "/acd4ef86-2258-4a54-89b2-1037db32041e"
-          (reference "R24") (unit 1)
+          (reference "R23") (unit 1)
         )
       )
@@
   (symbol (lib_id "Dragon32_MKII:R") (at 219.71 41.91 90) (unit 1)
     (in_bom yes) (on_board yes) (dnp no)
-    (property "Reference" "R23" (at 219.71 41.91 90)
+    (property "Reference" "R24" (at 219.71 41.91 90)
       (effects (font (size 1.27 1.27)))
     )
@@
       (project "Dragon32_MKII"
         (path "/acd4ef86-2258-4a54-89b2-1037db32041e"
-          (reference "R23") (unit 1)
+          (reference "R24") (unit 1)
         )
       )
@@
   (symbol (lib_id "Dragon32_MKII:R") (at 219.71 46.99 90) (unit 1)
     (in_bom yes) (on_board yes) (dnp no)
-    (property "Reference" "R21" (at 219.71 46.99 90)
+    (property "Reference" "R20" (at 219.71 46.99 90)
       (effects (font (size 1.27 1.27)))
     )
@@
       (project "Dragon32_MKII"
         (path "/acd4ef86-2258-4a54-89b2-1037db32041e"
-          (reference "R21") (unit 1)
+          (reference "R20") (unit 1)
         )
       )
@@
   (symbol (lib_id "Dragon32_MKII:R") (at 219.71 52.07 90) (unit 1)
     (in_bom yes) (on_board yes) (dnp no)
-    (property "Reference" "R20" (at 219.71 52.07 90)
+    (property "Reference" "R21" (at 219.71 52.07 90)
       (effects (font (size 1.27 1.27)))
     )
@@
       (project "Dragon32_MKII"
         (path "/acd4ef86-2258-4a54-89b2-1037db32041e"
-          (reference "R20") (unit 1)
+          (reference "R21") (unit 1)
         )
       )
@@
     )
   )
-  (symbol (lib_id "Dragon32_MKII:RELAY") (at 648.97 152.4 0) (unit 1)
-    (in_bom yes) (on_board yes) (dnp no)
-    (property "Reference" "RLA1" (at 652.78 142.24 0)
-      (effects (font (size 1.27 1.27)))
-    )
-    (property "Value" "RELAY" (at 651.51 142.24 0)
-      (effects (font (size 1.27 1.27)) hide)
-    )
-    (property "Footprint" "Dragon:OJS HM 10A Relay" (at 648.97 152.4 0)
-      (effects (font (size 1.524 1.524)) hide)
-    )
-    (property "Datasheet" "~" (at 648.97 152.4 0)
-      (effects (font (size 1.524 1.524)))
-    )
-    (pin "1")
-    (pin "2")
-    (pin "3")
-    (pin "4")
-    (instances
-      (project "Dragon32_MKII"
-        (path "/acd4ef86-2258-4a54-89b2-1037db32041e"
-          (reference "RLA1") (unit 1)
-        )
-      )
-    )
-  )
   (symbol (lib_id "Dragon32_MKII:R") (at 635 167.64 270) (unit 1)
     (in_bom yes) (on_board yes) (dnp no)
@@
     )
   )
-  (symbol (lib_id "Dragon32_MKII:DIODE") (at 638.81 152.4 90) (unit 1)
+  (symbol (lib_id "Dragon32_MKII:DIODE") (at 629.92 152.4 90) (unit 1)
     (in_bom yes) (on_board yes) (dnp no)
-    (property "Reference" "D1" (at 643.89 151.13 90)
+    (property "Reference" "D1" (at 635 151.13 90)
       (effects (font (size 1.27 1.27)) (justify left))
     )
-    (property "Value" "1N914" (at 647.7 153.67 90)
+    (property "Value" "1N914" (at 638.81 153.67 90)
       (effects (font (size 1.27 1.27)) (justify left))
     )
-    (property "Footprint" "Diode_THT:D_DO-35_SOD27_P12.70mm_Horizontal" (at 638.81 152.4 0)
+    (property "Footprint" "Diode_THT:D_DO-35_SOD27_P12.70mm_Horizontal" (at 629.92 152.4 0)
       (effects (font (size 1.524 1.524)) hide)
     )
-    (property "Datasheet" "~" (at 638.81 152.4 0)
+    (property "Datasheet" "~" (at 629.92 152.4 0)
       (effects (font (size 1.524 1.524)))
     )
@@
       (effects (font (size 1.27 1.27)) (justify left))
     )
-    (property "Footprint" "Capacitor_THT:CP_Radial_D5.0mm_P2.50mm" (at 568.96 378.46 0)
+    (property "Footprint" "Capacitor_THT:CP_Radial_Tantal_D5.5mm_P5.00mm" (at 568.96 378.46 0)
       (effects (font (size 1.524 1.524)) hide)
     )
@@
       (effects (font (size 1.27 1.27)) (justify left))
     )
-    (property "Footprint" "Capacitor_THT:CP_Radial_D5.0mm_P2.50mm" (at 568.96 344.17 0)
+    (property "Footprint" "Capacitor_THT:CP_Radial_Tantal_D6.0mm_P5.00mm" (at 568.96 344.17 0)
       (effects (font (size 1.524 1.524)) hide)
     )
@@
         )
       )
+    )
+  )
+  (symbol (lib_id "Relay:TIANBO-HJR-4102-L") (at 648.97 152.4 0) (mirror x) (unit 1)
+    (in_bom yes) (on_board yes) (dnp no)
+    (property "Reference" "RLA1" (at 659.892 153.5684 0)
+      (effects (font (size 1.27 1.27)) (justify right))
+    )
+    (property "Value" "SPDT" (at 659.892 151.257 0)
+      (effects (font (size 1.27 1.27)) (justify right))
+    )
+    (property "Footprint" "Relay_THT:Relay_SPDT_HJR-4102" (at 621.03 153.67 0)
+      (effects (font (size 1.27 1.27)) hide)
+    )
+    (property "Datasheet" "https://cdn-reichelt.de/documents/datenblatt/C300/DS_HJR4102E.pdf" (at 648.97 152.4 0)
+      (effects (font (size 1.27 1.27)) hide)
+    )
+    (pin "1")
+    (pin "12")
+    (pin "5")
+    (pin "6")
+    (pin "7")
+    (pin "8")
+    (instances
+      (project "Dragon32_MKII"
+        (path "/acd4ef86-2258-4a54-89b2-1037db32041e"
+          (reference "RLA1") (unit 1)
+        )
+      )
+      (project "dragon64"
+        (path "/e63e39d7-6ac0-4ffd-8aa3-1841a4541b55/00000000-0000-0000-0000-000060168bb0"
+          (reference "RLA1") (unit 1)
+        )
+      )

Commit message: fix z1 z2 wiring
Connections:
- net at IC15.29 (Z1): now also R24.1; no longer R23.1
- net at IC15.30 (Z2): now also R23.1; no longer R24.1
Changed lines of the file:
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@@
     (stroke (width 0) (type default))
   )
-  (wire (pts (xy 229.87 41.91) (xy 223.52 41.91))
-    (stroke (width 0) (type default))
-  )
   (bus (pts (xy 339.09 445.77) (xy 339.09 448.31))
     (stroke (width 0) (type default))
@@
     (stroke (width 0) (type default))
   )
-  (wire (pts (xy 229.87 39.37) (xy 223.52 39.37))
+  (wire (pts (xy 223.52 39.37) (xy 229.87 39.37))
     (stroke (width 0) (type default))
   )
@@
     (stroke (width 0) (type default))
   )
+  (wire (pts (xy 223.52 41.91) (xy 229.87 41.91))
+    (stroke (width 0) (type default))
+  )
   (bus (pts (xy 518.16 88.9) (xy 518.16 91.44))
     (stroke (width 0) (type default))
@@
     (effects (font (size 1.27 1.27)) (justify left bottom))
   )
-  (label "Z1" (at 226.06 39.37 0) (fields_autoplaced)
-    (effects (font (size 1.27 1.27)) (justify left bottom))
-  )
   (label "A2" (at 300.99 162.56 0) (fields_autoplaced)
     (effects (font (size 1.27 1.27)) (justify left bottom))
@@
     (effects (font (size 1.27 1.27)) (justify left bottom))
   )
+  (label "Z1" (at 226.06 41.91 0) (fields_autoplaced)
+    (effects (font (size 1.27 1.27)) (justify left bottom))
+  )
   (label "KB0" (at 584.2 63.5 0) (fields_autoplaced)
     (effects (font (size 1.27 1.27)) (justify left bottom))
@@
     (effects (font (size 1.27 1.27)) (justify left bottom))
   )
-  (label "Z2" (at 226.06 41.91 0) (fields_autoplaced)
-    (effects (font (size 1.27 1.27)) (justify left bottom))
-  )
   (label "Z5" (at 160.02 511.81 0) (fields_autoplaced)
     (effects (font (size 1.27 1.27)) (justify left bottom))
@@
     (effects (font (size 1.27 1.27)) (justify left bottom))
   )
+  (label "Z2" (at 226.06 39.37 0) (fields_autoplaced)
+    (effects (font (size 1.27 1.27)) (justify left bottom))
+  )
   (label "Z2" (at 220.98 440.69 0) (fields_autoplaced)
     (effects (font (size 1.27 1.27)) (justify left bottom))
@@
     )
   )
-  (symbol (lib_id "Dragon32_MKII:R") (at 219.71 39.37 90) (unit 1)
-    (in_bom yes) (on_board yes) (dnp no)
-    (property "Reference" "R23" (at 219.71 39.37 90)
-      (effects (font (size 1.27 1.27)))
-    )
-    (property "Value" "22R" (at 228.6 38.1 90)
-      (effects (font (size 1.27 1.27)) (justify left) hide)
-    )
-    (property "Footprint" "Dragon:R_Axial_DIN0207_L6.3mm_D2.5mm_P12.7mm_Horizontal" (at 219.71 41.148 90)
-      (effects (font (size 0.762 0.762)) hide)
-    )
-    (property "Datasheet" "~" (at 219.71 39.37 0)
-      (effects (font (size 0.762 0.762)))
-    )
-    (pin "1")
-    (pin "2")
-    (instances
-      (project "Dragon32_MKII"
-        (path "/acd4ef86-2258-4a54-89b2-1037db32041e"
-          (reference "R23") (unit 1)
-        )
-      )
-    )
-  )
-  (symbol (lib_id "Dragon32_MKII:R") (at 219.71 41.91 90) (unit 1)
-    (in_bom yes) (on_board yes) (dnp no)
-    (property "Reference" "R24" (at 219.71 41.91 90)
-      (effects (font (size 1.27 1.27)))
-    )
-    (property "Value" "22R" (at 228.6 40.64 90)
-      (effects (font (size 1.27 1.27)) (justify left) hide)
-    )
-    (property "Footprint" "Dragon:R_Axial_DIN0207_L6.3mm_D2.5mm_P12.7mm_Horizontal" (at 219.71 43.688 90)
-      (effects (font (size 0.762 0.762)) hide)
-    )
-    (property "Datasheet" "~" (at 219.71 41.91 0)
-      (effects (font (size 0.762 0.762)))
-    )
-    (pin "1")
-    (pin "2")
-    (instances
-      (project "Dragon32_MKII"
-        (path "/acd4ef86-2258-4a54-89b2-1037db32041e"
-          (reference "R24") (unit 1)
-        )
-      )
-    )
-  )
   (symbol (lib_id "Dragon32_MKII:R") (at 219.71 44.45 90) (unit 1)
     (in_bom yes) (on_board yes) (dnp no)
@@
     )
   )
+  (symbol (lib_id "Dragon32_MKII:R") (at 219.71 41.91 90) (unit 1)
+    (in_bom yes) (on_board yes) (dnp no)
+    (property "Reference" "R23" (at 219.71 41.91 90)
+      (effects (font (size 1.27 1.27)))
+    )
+    (property "Value" "22R" (at 228.6 40.64 90)
+      (effects (font (size 1.27 1.27)) (justify left) hide)
+    )
+    (property "Footprint" "Dragon:R_Axial_DIN0207_L6.3mm_D2.5mm_P12.7mm_Horizontal" (at 219.71 43.688 90)
+      (effects (font (size 0.762 0.762)) hide)
+    )
+    (property "Datasheet" "~" (at 219.71 41.91 0)
+      (effects (font (size 0.762 0.762)))
+    )
+    (pin "1")
+    (pin "2")
+    (instances
+      (project "Dragon32_MKII"
+        (path "/acd4ef86-2258-4a54-89b2-1037db32041e"
+          (reference "R23") (unit 1)
+        )
+      )
+    )
+  )
   (symbol (lib_id "Device:C_Small") (at 697.23 118.11 180) (unit 1)
     (in_bom yes) (on_board yes) (dnp no) (fields_autoplaced)
@@
         )
       )
+    )
+  )
+  (symbol (lib_id "Dragon32_MKII:R") (at 219.71 39.37 90) (unit 1)
+    (in_bom yes) (on_board yes) (dnp no)
+    (property "Reference" "R24" (at 219.71 39.37 90)
+      (effects (font (size 1.27 1.27)))
+    )
+    (property "Value" "22R" (at 228.6 38.1 90)
+      (effects (font (size 1.27 1.27)) (justify left) hide)
+    )
+    (property "Footprint" "Dragon:R_Axial_DIN0207_L6.3mm_D2.5mm_P12.7mm_Horizontal" (at 219.71 41.148 90)
+      (effects (font (size 0.762 0.762)) hide)
+    )
+    (property "Datasheet" "~" (at 219.71 39.37 0)
+      (effects (font (size 0.762 0.762)))
+    )
+    (pin "1")
+    (pin "2")
+    (instances
+      (project "Dragon32_MKII"
+        (path "/acd4ef86-2258-4a54-89b2-1037db32041e"
+          (reference "R24") (unit 1)
+        )
+      )
